File: elec/layout/default/hello-world.kicad_pcb (KiCad board)
At the start: 2 copper layers, 225.7 x 100.8 mm, 0 parts

Commit message: initial build
Parts:
- added C1: 25V 1uF X5R ±10% 0402 Multilayer Ceramic Capacitors MLCC - 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, lib:C0402, F.Cu at (113.2, 107.9)
- added C10: 25V 1uF X5R ±10% 0402 Multilayer Ceramic Capacitors MLCC - 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, lib:C0402, F.Cu at (125.8, 145.4)
- added C11: 25V 1uF X5R ±10% 0402 Multilayer Ceramic Capacitors MLCC - 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, lib:C0402, F.Cu at (123.6, 145.4)
- added C12: 25V 1uF X5R ±10% 0402 Multilayer Ceramic Capacitors MLCC - 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, lib:C0402, F.Cu at (122.5, 145.4)
- added C13: 25V 1uF X5R ±10% 0402 Multilayer Ceramic Capacitors MLCC - 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, lib:C0402, F.Cu at (113.2, 105.8)
- added C14: 25V 1uF X5R ±10% 0402 Multilayer Ceramic Capacitors MLCC - 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, lib:C0402, F.Cu at (124.7, 145.4)
- added C2: 16V 100nF X7R ±10% 0402 Multilayer Ceramic Capacitors MLCC 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, lib:C0402, F.Cu at (117.8, 167.1)
- added C3: 25V 10uF X5R ±10% 0805 Multilayer Ceramic Capacitors MLCC -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, lib:C0805, F.Cu at (119.3, 167.2)
- added C4: 25V 10uF X5R ±10% 0805 Multilayer Ceramic Capacitors MLCC -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, lib:C0805, F.Cu at (121.4, 167.2)
- added C5: 25V 1uF X5R ±10% 0402 Multilayer Ceramic Capacitors MLCC - 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, lib:C0402, F.Cu at (113.2, 106.8)
- added C6: 25V 1uF X5R ±10% 0402 Multilayer Ceramic Capacitors MLCC - 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, lib:C0402, F.Cu at (119.4, 145.4)
- added C7: 25V 1uF X5R ±10% 0402 Multilayer Ceramic Capacitors MLCC - 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, lib:C0402, F.Cu at (113.2, 104.8)
- added C8: 25V 1uF X5R ±10% 0402 Multilayer Ceramic Capacitors MLCC - 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, lib:C0402, F.Cu at (121.5, 145.4)
- added C9: 25V 1uF X5R ±10% 0402 Multilayer Ceramic Capacitors MLCC - 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, lib:C0402, F.Cu at (120.4, 145.4)
- added FID1: Fiducial_1.5mm_Mask3mm, Fiducial:Fiducial_1.5mm_Mask3mm, F.Cu at (139.5, 173.0)
- added FID2: Fiducial_1.5mm_Mask3mm, Fiducial:Fiducial_1.5mm_Mask3mm, F.Cu at (48.2, 173.2)
- added FID3: Fiducial_1.5mm_Mask3mm, Fiducial:Fiducial_1.5mm_Mask3mm, F.Cu at (48.5, 92.0)
- added FID4: Fiducial_1.5mm_Mask3mm, Fiducial:Fiducial_1.5mm_Mask3mm, F.Cu at (139.0, 93.0)
- added LED1: ?, lib:LED0402-RD_ORANGE, F.Cu at (102.7, 131.2)
- added LED10: ?, lib:LED0402-RD_ORANGE, F.Cu at (57.0, 135.7)
- added LED100: ?, lib:LED0402-RD_ORANGE, F.Cu at (100.1, 101.1)
- added LED101: ?, lib:LED0402-RD_ORANGE, F.Cu at (92.6, 114.4)
- added LED102: ?, lib:LED0402-RD_ORANGE, F.Cu at (95.1, 96.0)
- added LED103: ?, lib:LED0402-RD_ORANGE, F.Cu at (97.6, 109.0)
- added LED104: ?, lib:LED0402-RD_ORANGE, F.Cu at (102.7, 103.7)
- added LED105: ?, lib:LED0402-RD_ORANGE, F.Cu at (92.6, 93.0)
- added LED106: ?, lib:LED0402-RD_ORANGE, F.Cu at (90.0, 98.3)
- added LED107: ?, lib:LED0402-RD_ORANGE, F.Cu at (105.2, 95.7)
- added LED108: ?, lib:LED0402-RD_ORANGE, F.Cu at (95.1, 109.0)
- added LED109: ?, lib:LED0402-RD_ORANGE, F.Cu at (105.2, 114.4)
- added LED11: ?, lib:LED0402-RD_ORANGE, F.Cu at (97.1, 135.7)
- added LED110: ?, lib:LED0402-RD_ORANGE, F.Cu at (100.2, 114.4)
- added LED111: ?, lib:LED0402-RD_ORANGE, F.Cu at (97.6, 98.3)
- added LED112: ?, lib:LED0402-RD_ORANGE, F.Cu at (90.0, 93.1)
- added LED113: ?, lib:LED0402-RD_ORANGE, F.Cu at (84.9, 98.3)
- added LED114: ?, lib:LED0402-RD_ORANGE, F.Cu at (95.1, 106.3)
- added LED115: ?, lib:LED0402-RD_ORANGE, F.Cu at (84.9, 106.3)
- added LED116: ?, lib:LED0402-RD_ORANGE, F.Cu at (100.2, 103.7)
- added LED117: ?, lib:LED0402-RD_ORANGE, F.Cu at (84.9, 103.7)
- added LED118: ?, lib:LED0402-RD_ORANGE, F.Cu at (105.2, 98.3)
- added LED119: ?, lib:LED0402-RD_ORANGE, F.Cu at (105.2, 106.3)
- added LED12: ?, lib:LED0402-RD_ORANGE, F.Cu at (99.3, 134.0)
- added LED120: ?, lib:LED0402-RD_ORANGE, F.Cu at (105.2, 111.7)
- added LED121: ?, lib:LED0402-RD_ORANGE, F.Cu at (90.0, 109.1)
- added LED122: ?, lib:LED0402-RD_ORANGE, F.Cu at (99.9, 109.0)
- added LED123: ?, lib:LED0402-RD_ORANGE, F.Cu at (95.1, 93.0)
- added LED124: ?, lib:LED0402-RD_ORANGE, F.Cu at (102.7, 93.0)
- added LED125: ?, lib:LED0402-RD_ORANGE, F.Cu at (87.6, 109.0)
- added LED126: ?, lib:LED0402-RD_ORANGE, F.Cu at (102.7, 114.4)
- added LED127: ?, lib:LED0402-RD_ORANGE, F.Cu at (105.2, 93.0)
- added LED128: ?, lib:LED0402-RD_ORANGE, F.Cu at (87.4, 98.4)
- added LED129: ?, lib:LED0402-RD_ORANGE, F.Cu at (90.0, 103.7)
- added LED13: ?, lib:LED0402-RD_ORANGE, F.Cu at (110.6, 128.9)
- added LED130: ?, lib:LED0402-RD_ORANGE, F.Cu at (84.9, 114.4)
- added LED131: ?, lib:LED0402-RD_ORANGE, F.Cu at (95.1, 114.4)
- added LED132: ?, lib:LED0402-RD_ORANGE, F.Cu at (95.1, 103.7)
- added LED133: ?, lib:LED0402-RD_ORANGE, F.Cu at (97.6, 114.4)
- added LED134: ?, lib:LED0402-RD_ORANGE, F.Cu at (90.0, 101.0)
- added LED135: ?, lib:LED0402-RD_ORANGE, F.Cu at (95.1, 98.3)
- added LED136: ?, lib:LED0402-RD_ORANGE, F.Cu at (105.2, 103.7)
- added LED137: ?, lib:LED0402-RD_ORANGE, F.Cu at (105.2, 109.0)
- added LED138: ?, lib:LED0402-RD_ORANGE, F.Cu at (90.0, 114.4)
- added LED139: ?, lib:LED0402-RD_ORANGE, F.Cu at (92.6, 103.7)
- added LED14: ?, lib:LED0402-RD_ORANGE, F.Cu at (59.6, 133.5)
- added LED140: ?, lib:LED0402-RD_ORANGE, F.Cu at (90.0, 111.6)
- added LED141: ?, lib:LED0402-RD_ORANGE, F.Cu at (100.2, 93.0)
- added LED142: ?, lib:LED0402-RD_ORANGE, F.Cu at (84.9, 93.0)
- added LED143: ?, lib:LED0402-RD_ORANGE, F.Cu at (100.2, 98.3)
- added LED144: ?, lib:LED0402-RD_ORANGE, F.Cu at (84.9, 109.0)
- added LED15: ?, lib:LED0402-RD_ORANGE, F.Cu at (108.0, 128.9)
- added LED16: ?, lib:LED0402-RD_ORANGE, F.Cu at (135.1, 128.9)
- added LED17: ?, lib:LED0402-RD_ORANGE, F.Cu at (65.6, 135.7)
- added LED18: ?, lib:LED0402-RD_ORANGE, F.Cu at (121.0, 129.2)
- added LED19: ?, lib:LED0402-RD_ORANGE, F.Cu at (59.6, 138.0)
- added LED2: ?, lib:LED0402-RD_ORANGE, F.Cu at (52.9, 135.7)
- added LED20: ?, lib:LED0402-RD_ORANGE, F.Cu at (79.9, 130.5)
- added LED21: ?, lib:LED0402-RD_ORANGE, F.Cu at (112.0, 135.7)
- added LED22: ?, lib:LED0402-RD_ORANGE, F.Cu at (141.2, 128.9)
- added LED23: ?, lib:LED0402-RD_ORANGE, F.Cu at (47.7, 131.2)
- added LED24: ?, lib:LED0402-RD_ORANGE, F.Cu at (116.1, 128.9)
- added LED25: ?, lib:LED0402-RD_ORANGE, F.Cu at (99.3, 131.6)
- added LED26: ?, lib:LED0402-RD_ORANGE, F.Cu at (97.6, 138.0)
- added LED27: ?, lib:LED0402-RD_ORANGE, F.Cu at (137.0, 130.4)
- added LED28: ?, lib:LED0402-RD_ORANGE, F.Cu at (101.7, 135.7)
- added LED29: ?, lib:LED0402-RD_ORANGE, F.Cu at (106.5, 135.7)
- added LED3: ?, lib:LED0402-RD_ORANGE, F.Cu at (68.0, 138.0)
- added LED30: ?, lib:LED0402-RD_ORANGE, F.Cu at (118.8, 133.4)
- added LED31: ?, lib:LED0402-RD_ORANGE, F.Cu at (85.4, 130.5)
- added LED32: ?, lib:LED0402-RD_ORANGE, F.Cu at (59.6, 128.9)
- added LED33: ?, lib:LED0402-RD_ORANGE, F.Cu at (125.0, 128.9)
- added LED34: ?, lib:LED0402-RD_ORANGE, F.Cu at (103.2, 128.9)
- added LED35: ?, lib:LED0402-RD_ORANGE, F.Cu at (121.1, 131.5)
- added LED36: ?, lib:LED0402-RD_ORANGE, F.Cu at (110.5, 138.0)
- added LED37: ?, lib:LED0402-RD_ORANGE, F.Cu at (61.9, 128.9)
- added LED38: ?, lib:LED0402-RD_ORANGE, F.Cu at (132.4, 133.4)
- added LED39: ?, lib:LED0402-RD_ORANGE, F.Cu at (96.0, 131.2)
- added LED4: ?, lib:LED0402-RD_ORANGE, F.Cu at (83.8, 138.0)
- added LED40: ?, lib:LED0402-RD_ORANGE, F.Cu at (79.9, 135.8)
- added LED41: ?, lib:LED0402-RD_ORANGE, F.Cu at (132.4, 135.8)
- added LED42: ?, lib:LED0402-RD_ORANGE, F.Cu at (72.8, 128.9)
- added LED43: ?, lib:LED0402-RD_ORANGE, F.Cu at (129.9, 138.0)
- added LED44: ?, lib:LED0402-RD_ORANGE, F.Cu at (52.9, 128.9)
- added LED45: ?, lib:LED0402-RD_ORANGE, F.Cu at (75.4, 138.0)
- added LED46: ?, lib:LED0402-RD_ORANGE, F.Cu at (50.4, 134.7)
- added LED47: ?, lib:LED0402-RD_ORANGE, F.Cu at (141.2, 131.6)
- added LED48: ?, lib:LED0402-RD_ORANGE, F.Cu at (85.8, 133.0)
- added LED49: ?, lib:LED0402-RD_ORANGE, F.Cu at (96.5, 133.5)
- added LED5: ?, lib:LED0402-RD_ORANGE, F.Cu at (57.0, 131.2)
- added LED50: ?, lib:LED0402-RD_ORANGE, F.Cu at (81.1, 128.9)
- added LED51: ?, lib:LED0402-RD_ORANGE, F.Cu at (72.8, 138.0)
- added LED52: ?, lib:LED0402-RD_ORANGE, F.Cu at (61.9, 138.0)
- added LED53: ?, lib:LED0402-RD_ORANGE, F.Cu at (47.7, 138.0)
- added LED54: ?, lib:LED0402-RD_ORANGE, F.Cu at (102.1, 133.5)
- added LED55: ?, lib:LED0402-RD_ORANGE, F.Cu at (118.7, 128.9)
- added LED56: ?, lib:LED0402-RD_ORANGE, F.Cu at (95.6, 128.9)
- added LED57: ?, lib:LED0402-RD_ORANGE, F.Cu at (116.1, 133.5)
- added LED58: ?, lib:LED0402-RD_ORANGE, F.Cu at (125.0, 131.0)
- added LED59: ?, lib:LED0402-RD_ORANGE, F.Cu at (65.6, 131.2)
- added LED6: ?, lib:LED0402-RD_ORANGE, F.Cu at (70.2, 138.0)
- added LED60: ?, lib:LED0402-RD_ORANGE, F.Cu at (112.2, 133.5)
- added LED61: ?, lib:LED0402-RD_ORANGE, F.Cu at (112.0, 131.2)
- added LED62: ?, lib:LED0402-RD_ORANGE, F.Cu at (106.3, 133.5)
- added LED63: ?, lib:LED0402-RD_ORANGE, F.Cu at (141.2, 138.0)
- added LED64: ?, lib:LED0402-RD_ORANGE, F.Cu at (72.8, 135.7)
- added LED65: ?, lib:LED0402-RD_ORANGE, F.Cu at (106.4, 131.2)
- added LED66: ?, lib:LED0402-RD_ORANGE, F.Cu at (135.0, 138.0)
- added LED67: ?, lib:LED0402-RD_ORANGE, F.Cu at (132.4, 131.0)
- added LED68: ?, lib:LED0402-RD_ORANGE, F.Cu at (72.8, 133.5)
- added LED69: ?, lib:LED0402-RD_ORANGE, F.Cu at (52.9, 138.0)
- added LED7: ?, lib:LED0402-RD_ORANGE, F.Cu at (81.1, 138.0)
- added LED70: ?, lib:LED0402-RD_ORANGE, F.Cu at (137.6, 133.2)
- added LED71: ?, lib:LED0402-RD_ORANGE, F.Cu at (132.4, 128.9)
- added LED72: ?, lib:LED0402-RD_ORANGE, F.Cu at (125.0, 138.0)
- added LED73: ?, lib:LED0402-RD_ORANGE, F.Cu at (72.8, 131.2)
- added LED74: ?, lib:LED0402-RD_ORANGE, F.Cu at (132.4, 138.0)
- added LED75: ?, lib:LED0402-RD_ORANGE, F.Cu at (57.0, 138.0)
- added LED76: ?, lib:LED0402-RD_ORANGE, F.Cu at (83.7, 128.9)
- added LED77: ?, lib:LED0402-RD_ORANGE, F.Cu at (85.4, 135.8)
- added LED78: ?, lib:LED0402-RD_ORANGE, F.Cu at (65.6, 128.9)
- added LED79: ?, lib:LED0402-RD_ORANGE, F.Cu at (57.0, 128.9)
- added LED8: ?, lib:LED0402-RD_ORANGE, F.Cu at (116.1, 138.0)
- added LED80: ?, lib:LED0402-RD_ORANGE, F.Cu at (116.1, 135.7)
- added LED81: ?, lib:LED0402-RD_ORANGE, F.Cu at (79.6, 132.9)
- added LED82: ?, lib:LED0402-RD_ORANGE, F.Cu at (47.7, 128.9)
- added LED83: ?, lib:LED0402-RD_ORANGE, F.Cu at (52.9, 133.5)
- added LED84: ?, lib:LED0402-RD_ORANGE, F.Cu at (65.6, 133.5)
- added LED85: ?, lib:LED0402-RD_ORANGE, F.Cu at (125.0, 135.8)
- added LED86: ?, lib:LED0402-RD_ORANGE, F.Cu at (127.5, 138.0)
- added LED87: ?, lib:LED0402-RD_ORANGE, F.Cu at (77.7, 138.0)
- added LED88: ?, lib:LED0402-RD_ORANGE, F.Cu at (116.1, 131.2)
- added LED89: ?, lib:LED0402-RD_ORANGE, F.Cu at (121.0, 138.0)
- added LED9: ?, lib:LED0402-RD_ORANGE, F.Cu at (101.0, 138.0)
- added LED90: ?, lib:LED0402-RD_ORANGE, F.Cu at (52.9, 131.2)
- added LED91: ?, lib:LED0402-RD_ORANGE, F.Cu at (47.7, 133.5)
- added LED92: ?, lib:LED0402-RD_ORANGE, F.Cu at (107.9, 138.0)
- added LED93: ?, lib:LED0402-RD_ORANGE, F.Cu at (47.7, 135.7)
- added LED94: ?, lib:LED0402-RD_ORANGE, F.Cu at (119.8, 135.8)
- added LED95: ?, lib:LED0402-RD_ORANGE, F.Cu at (65.6, 138.0)
- added LED96: ?, lib:LED0402-RD_ORANGE, F.Cu at (141.2, 134.1)
- added LED97: ?, lib:LED0402-RD_ORANGE, F.Cu at (125.0, 133.3)
- added LED98: ?, lib:LED0402-RD_ORANGE, F.Cu at (137.2, 135.8)
- added LED99: ?, lib:LED0402-RD_ORANGE, F.Cu at (57.0, 133.5)
- added Q1: ?, lib:SOT-23-3_L2.9-W1.3-P1.90-LS2.4-BR, F.Cu at (116.8, 145.0)
- added Q2: ?, lib:SOT-23-3_L2.9-W1.3-P1.90-LS2.4-BR, F.Cu at (112.8, 110.7)
- added R1: 62.5mW Thick Film Resistors 50V ±100ppm/℃ ±1% 4.7kΩ 0402 Ch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, lib:R0402, F.Cu at (81.2, 168.6)
- added R10: 62.5mW Thick Film Resistors 50V ±100ppm/℃ ±1% 5.49kΩ 0402 C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, lib:R0402, F.Cu at (68.1, 139.1)
- added R100: 62.5mW Thick Film Resistors 50V ±100ppm/℃ ±1% 5.49kΩ 0402 C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, lib:R0402, F.Cu at (47.7, 136.8)
- added R101: 62.5mW Thick Film Resistors 50V ±100ppm/℃ ±1% 5.49kΩ 0402 C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, lib:R0402, F.Cu at (119.9, 136.8)
- added R102: 62.5mW Thick Film Resistors 50V ±100ppm/℃ ±1% 5.49kΩ 0402 C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, lib:R0402, F.Cu at (65.6, 139.1)
- added R103: 62.5mW Thick Film Resistors 50V ±100ppm/℃ ±1% 5.49kΩ 0402 C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, lib:R0402, F.Cu at (141.3, 135.2)
- added R104: 62.5mW Thick Film Resistors 50V ±100ppm/℃ ±1% 5.49kΩ 0402 C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, lib:R0402, F.Cu at (125.0, 134.4)
- added R105: 62.5mW Thick Film Resistors 50V ±100ppm/℃ ±1% 5.49kΩ 0402 C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, lib:R0402, F.Cu at (137.3, 136.8)
- added R106: 62.5mW Thick Film Resistors 50V ±100ppm/℃ ±1% 5.49kΩ 0402 C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, lib:R0402, F.Cu at (57.1, 134.5)
- added R107: 62.5mW Thick Film Resistors 50V ±100ppm/℃ ±1% 5.49kΩ 0402 C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, lib:R0402, F.Cu at (100.2, 102.2)
- added R108: 62.5mW Thick Film Resistors 50V ±100ppm/℃ ±1% 5.49kΩ 0402 C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, lib:R0402, F.Cu at (92.6, 115.4)
- added R109: 62.5mW Thick Film Resistors 50V ±100ppm/℃ ±1% 5.49kΩ 0402 C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, lib:R0402, F.Cu at (95.1, 97.0)
- added R11: 62.5mW Thick Film Resistors 50V ±100ppm/℃ ±1% 5.49kΩ 0402 C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, lib:R0402, F.Cu at (83.9, 139.1)
- added R110: 62.5mW Thick Film Resistors 50V ±100ppm/℃ ±1% 5.49kΩ 0402 C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, lib:R0402, F.Cu at (97.6, 110.1)
- added R111: 62.5mW Thick Film Resistors 50V ±100ppm/℃ ±1% 5.49kΩ 0402 C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, lib:R0402, F.Cu at (102.8, 104.7)
- added R112: 62.5mW Thick Film Resistors 50V ±100ppm/℃ ±1% 5.49kΩ 0402 C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, lib:R0402, F.Cu at (92.6, 94.1)
- added R113: 62.5mW Thick Film Resistors 50V ±100ppm/℃ ±1% 5.49kΩ 0402 C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, lib:R0402, F.Cu at (90.1, 99.4)
- added R114: 62.5mW Thick Film Resistors 50V ±100ppm/℃ ±1% 5.49kΩ 0402 C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, lib:R0402, F.Cu at (105.2, 96.7)
- added R115: 62.5mW Thick Film Resistors 50V ±100ppm/℃ ±1% 5.49kΩ 0402 C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, lib:R0402, F.Cu at (95.1, 110.1)
- added R116: 62.5mW Thick Film Resistors 50V ±100ppm/℃ ±1% 5.49kΩ 0402 C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, lib:R0402, F.Cu at (105.2, 115.4)
- added R117: 62.5mW Thick Film Resistors 50V ±100ppm/℃ ±1% 5.49kΩ 0402 C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, lib:R0402, F.Cu at (100.2, 115.4)
- added R118: 62.5mW Thick Film Resistors 50V ±100ppm/℃ ±1% 5.49kΩ 0402 C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, lib:R0402, F.Cu at (97.7, 99.4)
- added R119: 62.5mW Thick Film Resistors 50V ±100ppm/℃ ±1% 5.49kΩ 0402 C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, lib:R0402, F.Cu at (90.1, 94.2)
- added R12: 62.5mW Thick Film Resistors 50V ±100ppm/℃ ±1% 5.49kΩ 0402 C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, lib:R0402, F.Cu at (57.1, 132.2)
- added R120: 62.5mW Thick Film Resistors 50V ±100ppm/℃ ±1% 5.49kΩ 0402 C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, lib:R0402, F.Cu at (84.9, 99.4)
- added R121: 62.5mW Thick Film Resistors 50V ±100ppm/℃ ±1% 5.49kΩ 0402 C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, lib:R0402, F.Cu at (95.1, 107.4)
- added R122: 62.5mW Thick Film Resistors 50V ±100ppm/℃ ±1% 5.49kΩ 0402 C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, lib:R0402, F.Cu at (84.9, 107.4)
- added R123: 62.5mW Thick Film Resistors 50V ±100ppm/℃ ±1% 5.49kΩ 0402 C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, lib:R0402, F.Cu at (100.2, 104.7)
- added R124: 62.5mW Thick Film Resistors 50V ±100ppm/℃ ±1% 5.49kΩ 0402 C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, lib:R0402, F.Cu at (84.9, 104.7)
- added R125: 62.5mW Thick Film Resistors 50V ±100ppm/℃ ±1% 5.49kΩ 0402 C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, lib:R0402, F.Cu at (105.2, 99.4)
- added R126: 62.5mW Thick Film Resistors 50V ±100ppm/℃ ±1% 5.49kΩ 0402 C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, lib:R0402, F.Cu at (105.2, 107.4)
- added R127: 62.5mW Thick Film Resistors 50V ±100ppm/℃ ±1% 5.49kΩ 0402 C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, lib:R0402, F.Cu at (105.2, 112.7)
- added R128: 62.5mW Thick Film Resistors 50V ±100ppm/℃ ±1% 5.49kΩ 0402 C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, lib:R0402, F.Cu at (90.1, 110.2)
- added R129: 62.5mW Thick Film Resistors 50V ±100ppm/℃ ±1% 5.49kΩ 0402 C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, lib:R0402, F.Cu at (99.9, 110.1)
- added R13: 62.5mW Thick Film Resistors 50V ±100ppm/℃ ±1% 5.49kΩ 0402 C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, lib:R0402, F.Cu at (70.3, 139.1)
- added R130: 62.5mW Thick Film Resistors 50V ±100ppm/℃ ±1% 5.49kΩ 0402 C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, lib:R0402, F.Cu at (95.1, 94.1)
- added R131: 62.5mW Thick Film Resistors 50V ±100ppm/℃ ±1% 5.49kΩ 0402 C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, lib:R0402, F.Cu at (102.8, 94.1)
- added R132: 62.5mW Thick Film Resistors 50V ±100ppm/℃ ±1% 5.49kΩ 0402 C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, lib:R0402, F.Cu at (87.7, 110.1)
- added R133: 62.5mW Thick Film Resistors 50V ±100ppm/℃ ±1% 5.49kΩ 0402 C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, lib:R0402, F.Cu at (102.8, 115.4)
- added R134: 62.5mW Thick Film Resistors 50V ±100ppm/℃ ±1% 5.49kΩ 0402 C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, lib:R0402, F.Cu at (105.2, 94.1)
- added R135: 62.5mW Thick Film Resistors 50V ±100ppm/℃ ±1% 5.49kΩ 0402 C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, lib:R0402, F.Cu at (87.5, 99.4)
- added R136: 62.5mW Thick Film Resistors 50V ±100ppm/℃ ±1% 5.49kΩ 0402 C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, lib:R0402, F.Cu at (90.1, 104.7)
- added R137: 62.5mW Thick Film Resistors 50V ±100ppm/℃ ±1% 5.49kΩ 0402 C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, lib:R0402, F.Cu at (85.0, 115.4)
- added R138: 62.5mW Thick Film Resistors 50V ±100ppm/℃ ±1% 5.49kΩ 0402 C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, lib:R0402, F.Cu at (95.1, 115.4)
- added R139: 62.5mW Thick Film Resistors 50V ±100ppm/℃ ±1% 5.49kΩ 0402 C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, lib:R0402, F.Cu at (95.1, 104.7)
- added R14: 62.5mW Thick Film Resistors 50V ±100ppm/℃ ±1% 5.49kΩ 0402 C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, lib:R0402, F.Cu at (81.2, 139.1)
- added R140: 62.5mW Thick Film Resistors 50V ±100ppm/℃ ±1% 5.49kΩ 0402 C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, lib:R0402, F.Cu at (97.7, 115.4)
- added R141: 62.5mW Thick Film Resistors 50V ±100ppm/℃ ±1% 5.49kΩ 0402 C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, lib:R0402, F.Cu at (90.1, 102.1)
- added R142: 62.5mW Thick Film Resistors 50V ±100ppm/℃ ±1% 5.49kΩ 0402 C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, lib:R0402, F.Cu at (95.1, 99.4)
- added R143: 62.5mW Thick Film Resistors 50V ±100ppm/℃ ±1% 5.49kΩ 0402 C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, lib:R0402, F.Cu at (105.2, 104.7)
- added R144: 62.5mW Thick Film Resistors 50V ±100ppm/℃ ±1% 5.49kΩ 0402 C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, lib:R0402, F.Cu at (105.2, 110.1)
- added R145: 62.5mW Thick Film Resistors 50V ±100ppm/℃ ±1% 5.49kΩ 0402 C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, lib:R0402, F.Cu at (90.1, 115.4)
- added R146: 62.5mW Thick Film Resistors 50V ±100ppm/℃ ±1% 5.49kΩ 0402 C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, lib:R0402, F.Cu at (92.6, 104.7)
- added R147: 62.5mW Thick Film Resistors 50V ±100ppm/℃ ±1% 5.49kΩ 0402 C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, lib:R0402, F.Cu at (90.1, 112.6)
- added R148: 62.5mW Thick Film Resistors 50V ±100ppm/℃ ±1% 5.49kΩ 0402 C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, lib:R0402, F.Cu at (100.2, 94.1)
- added R149: 62.5mW Thick Film Resistors 50V ±100ppm/℃ ±1% 5.49kΩ 0402 C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, lib:R0402, F.Cu at (84.9, 94.1)
- added R15: 62.5mW Thick Film Resistors 50V ±100ppm/℃ ±1% 5.49kΩ 0402 C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, lib:R0402, F.Cu at (116.1, 139.1)
- added R150: 62.5mW Thick Film Resistors 50V ±100ppm/℃ ±1% 5.49kΩ 0402 C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, lib:R0402, F.Cu at (100.2, 99.4)
- added R151: 62.5mW Thick Film Resistors 50V ±100ppm/℃ ±1% 5.49kΩ 0402 C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, lib:R0402, F.Cu at (85.0, 110.1)
- added R16: 62.5mW Thick Film Resistors 50V ±100ppm/℃ ±1% 5.49kΩ 0402 C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, lib:R0402, F.Cu at (101.1, 139.1)
- added R17: 62.5mW Thick Film Resistors 50V ±100ppm/℃ ±1% 5.49kΩ 0402 C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, lib:R0402, F.Cu at (57.1, 136.8)
- added R18: 62.5mW Thick Film Resistors 50V ±100ppm/℃ ±1% 5.49kΩ 0402 C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, lib:R0402, F.Cu at (97.2, 136.8)
- added R19: 62.5mW Thick Film Resistors 50V ±100ppm/℃ ±1% 5.49kΩ 0402 C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, lib:R0402, F.Cu at (99.4, 135.1)
- added R2: 62.5mW Thick Film Resistors 50V ±100ppm/℃ ±1% 4.7kΩ 0402 Ch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, lib:R0402, F.Cu at (84.2, 168.5)
- added R20: 62.5mW Thick Film Resistors 50V ±100ppm/℃ ±1% 5.49kΩ 0402 C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, lib:R0402, F.Cu at (110.6, 130.0)
- added R21: 62.5mW Thick Film Resistors 50V ±100ppm/℃ ±1% 5.49kΩ 0402 C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, lib:R0402, F.Cu at (59.6, 134.5)
- added R22: 62.5mW Thick Film Resistors 50V ±100ppm/℃ ±1% 5.49kΩ 0402 C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, lib:R0402, F.Cu at (108.1, 130.0)
- added R23: 62.5mW Thick Film Resistors 50V ±100ppm/℃ ±1% 5.49kΩ 0402 C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, lib:R0402, F.Cu at (135.2, 130.0)
- added R24: 62.5mW Thick Film Resistors 50V ±100ppm/℃ ±1% 5.49kΩ 0402 C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, lib:R0402, F.Cu at (65.6, 136.8)
- added R25: 62.5mW Thick Film Resistors 50V ±100ppm/℃ ±1% 5.49kΩ 0402 C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, lib:R0402, F.Cu at (121.1, 130.2)
- added R26: 62.5mW Thick Film Resistors 50V ±100ppm/℃ ±1% 5.49kΩ 0402 C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, lib:R0402, F.Cu at (59.6, 139.1)
- added R27: 62.5mW Thick Film Resistors 50V ±100ppm/℃ ±1% 5.49kΩ 0402 C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, lib:R0402, F.Cu at (79.9, 131.5)
- added R28: 62.5mW Thick Film Resistors 50V ±100ppm/℃ ±1% 5.49kΩ 0402 C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, lib:R0402, F.Cu at (112.0, 136.8)
- added R29: 62.5mW Thick Film Resistors 50V ±100ppm/℃ ±1% 5.49kΩ 0402 C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, lib:R0402, F.Cu at (141.3, 130.0)
- added R3: 62.5mW Thick Film Resistors 50V ±100ppm/℃ ±1% 10kΩ 0402 Chi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, lib:R0402, F.Cu at (118.4, 164.4)
- added R30: 62.5mW Thick Film Resistors 50V ±100ppm/℃ ±1% 5.49kΩ 0402 C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, lib:R0402, F.Cu at (47.7, 132.2)
- added R31: 62.5mW Thick Film Resistors 50V ±100ppm/℃ ±1% 5.49kΩ 0402 C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, lib:R0402, F.Cu at (116.1, 130.0)
- added R32: 62.5mW Thick Film Resistors 50V ±100ppm/℃ ±1% 5.49kΩ 0402 C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, lib:R0402, F.Cu at (99.4, 132.7)
- added R33: 62.5mW Thick Film Resistors 50V ±100ppm/℃ ±1% 5.49kΩ 0402 C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, lib:R0402, F.Cu at (97.6, 139.1)
- added R34: 62.5mW Thick Film Resistors 50V ±100ppm/℃ ±1% 5.49kΩ 0402 C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, lib:R0402, F.Cu at (137.0, 131.5)
- added R35: 62.5mW Thick Film Resistors 50V ±100ppm/℃ ±1% 5.49kΩ 0402 C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, lib:R0402, F.Cu at (101.7, 136.8)
- added R36: 62.5mW Thick Film Resistors 50V ±100ppm/℃ ±1% 5.49kΩ 0402 C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, lib:R0402, F.Cu at (106.5, 136.8)
- added R37: 62.5mW Thick Film Resistors 50V ±100ppm/℃ ±1% 5.49kΩ 0402 C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, lib:R0402, F.Cu at (118.9, 134.5)
- added R38: 62.5mW Thick Film Resistors 50V ±100ppm/℃ ±1% 5.49kΩ 0402 C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, lib:R0402, F.Cu at (85.4, 131.6)
- added R39: 62.5mW Thick Film Resistors 50V ±100ppm/℃ ±1% 5.49kΩ 0402 C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, lib:R0402, F.Cu at (59.6, 130.0)
- added R4: 62.5mW Thick Film Resistors 50V ±100ppm/℃ ±1% 4.7kΩ 0402 Ch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, lib:R0402, F.Cu at (114.4, 145.8)
- added R40: 62.5mW Thick Film Resistors 50V ±100ppm/℃ ±1% 5.49kΩ 0402 C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, lib:R0402, F.Cu at (125.0, 130.0)
- added R41: 62.5mW Thick Film Resistors 50V ±100ppm/℃ ±1% 5.49kΩ 0402 C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, lib:R0402, F.Cu at (103.2, 130.0)
- added R42: 62.5mW Thick Film Resistors 50V ±100ppm/℃ ±1% 5.49kΩ 0402 C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, lib:R0402, F.Cu at (121.2, 132.6)
- added R43: 62.5mW Thick Film Resistors 50V ±100ppm/℃ ±1% 5.49kΩ 0402 C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, lib:R0402, F.Cu at (110.5, 139.1)
- added R44: 62.5mW Thick Film Resistors 50V ±100ppm/℃ ±1% 5.49kΩ 0402 C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, lib:R0402, F.Cu at (61.9, 130.0)
- added R45: 62.5mW Thick Film Resistors 50V ±100ppm/℃ ±1% 5.49kΩ 0402 C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, lib:R0402, F.Cu at (132.4, 134.5)
- added R46: 62.5mW Thick Film Resistors 50V ±100ppm/℃ ±1% 5.49kΩ 0402 C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, lib:R0402, F.Cu at (96.1, 132.2)
- added R47: 62.5mW Thick Film Resistors 50V ±100ppm/℃ ±1% 5.49kΩ 0402 C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, lib:R0402, F.Cu at (80.0, 136.8)
- added R48: 62.5mW Thick Film Resistors 50V ±100ppm/℃ ±1% 5.49kΩ 0402 C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, lib:R0402, F.Cu at (132.4, 136.8)
- added R49: 62.5mW Thick Film Resistors 50V ±100ppm/℃ ±1% 5.49kΩ 0402 C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, lib:R0402, F.Cu at (72.9, 130.0)
- added R5: 62.5mW Thick Film Resistors 50V ±100ppm/℃ ±1% 4.7kΩ 0402 Ch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, lib:R0402, F.Cu at (113.4, 145.8)
- added R50: 62.5mW Thick Film Resistors 50V ±100ppm/℃ ±1% 5.49kΩ 0402 C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, lib:R0402, F.Cu at (129.9, 139.1)
- added R51: 62.5mW Thick Film Resistors 50V ±100ppm/℃ ±1% 5.49kΩ 0402 C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, lib:R0402, F.Cu at (52.9, 130.0)
- added R52: 62.5mW Thick Film Resistors 50V ±100ppm/℃ ±1% 5.49kΩ 0402 C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, lib:R0402, F.Cu at (75.4, 139.1)
- added R53: 62.5mW Thick Film Resistors 50V ±100ppm/℃ ±1% 5.49kΩ 0402 C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, lib:R0402, F.Cu at (50.3, 133.6)
- added R54: 62.5mW Thick Film Resistors 50V ±100ppm/℃ ±1% 5.49kΩ 0402 C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, lib:R0402, F.Cu at (141.3, 132.6)
- added R55: 62.5mW Thick Film Resistors 50V ±100ppm/℃ ±1% 5.49kΩ 0402 C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, lib:R0402, F.Cu at (85.8, 134.1)
- added R56: 62.5mW Thick Film Resistors 50V ±100ppm/℃ ±1% 5.49kΩ 0402 C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, lib:R0402, F.Cu at (96.5, 134.5)
- added R57: 62.5mW Thick Film Resistors 50V ±100ppm/℃ ±1% 5.49kΩ 0402 C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, lib:R0402, F.Cu at (81.2, 130.0)
- added R58: 62.5mW Thick Film Resistors 50V ±100ppm/℃ ±1% 5.49kΩ 0402 C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, lib:R0402, F.Cu at (72.9, 139.1)
- added R59: 62.5mW Thick Film Resistors 50V ±100ppm/℃ ±1% 5.49kΩ 0402 C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, lib:R0402, F.Cu at (62.0, 139.1)
- added R6: 62.5mW Thick Film Resistors 50V ±100ppm/℃ ±1% 4.7kΩ 0402 Ch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, lib:R0402, F.Cu at (113.4, 113.1)
- added R60: 62.5mW Thick Film Resistors 50V ±100ppm/℃ ±1% 5.49kΩ 0402 C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, lib:R0402, F.Cu at (47.7, 139.1)
- added R61: 62.5mW Thick Film Resistors 50V ±100ppm/℃ ±1% 5.49kΩ 0402 C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, lib:R0402, F.Cu at (102.1, 134.5)
- added R62: 62.5mW Thick Film Resistors 50V ±100ppm/℃ ±1% 5.49kΩ 0402 C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, lib:R0402, F.Cu at (118.8, 130.0)
- added R63: 62.5mW Thick Film Resistors 50V ±100ppm/℃ ±1% 5.49kΩ 0402 C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, lib:R0402, F.Cu at (95.6, 130.0)
- added R64: 62.5mW Thick Film Resistors 50V ±100ppm/℃ ±1% 5.49kΩ 0402 C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, lib:R0402, F.Cu at (116.1, 134.5)
- added R65: 62.5mW Thick Film Resistors 50V ±100ppm/℃ ±1% 5.49kΩ 0402 C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, lib:R0402, F.Cu at (125.0, 132.0)
- added R66: 62.5mW Thick Film Resistors 50V ±100ppm/℃ ±1% 5.49kΩ 0402 C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, lib:R0402, F.Cu at (65.6, 132.2)
- added R67: 62.5mW Thick Film Resistors 50V ±100ppm/℃ ±1% 5.49kΩ 0402 C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, lib:R0402, F.Cu at (112.2, 134.5)
- added R68: 62.5mW Thick Film Resistors 50V ±100ppm/℃ ±1% 5.49kΩ 0402 C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, lib:R0402, F.Cu at (112.1, 132.2)
- added R69: 62.5mW Thick Film Resistors 50V ±100ppm/℃ ±1% 5.49kΩ 0402 C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, lib:R0402, F.Cu at (106.4, 134.5)
- added R7: 62.5mW Thick Film Resistors 50V ±100ppm/℃ ±1% 4.7kΩ 0402 Ch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, lib:R0402, F.Cu at (113.4, 114.3)
- added R70: 62.5mW Thick Film Resistors 50V ±100ppm/℃ ±1% 5.49kΩ 0402 C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, lib:R0402, F.Cu at (141.3, 139.1)
- added R71: 62.5mW Thick Film Resistors 50V ±100ppm/℃ ±1% 5.49kΩ 0402 C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, lib:R0402, F.Cu at (72.9, 136.8)
- added R72: 62.5mW Thick Film Resistors 50V ±100ppm/℃ ±1% 5.49kΩ 0402 C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, lib:R0402, F.Cu at (106.5, 132.2)
- added R73: 62.5mW Thick Film Resistors 50V ±100ppm/℃ ±1% 5.49kΩ 0402 C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, lib:R0402, F.Cu at (135.1, 139.1)
- added R74: 62.5mW Thick Film Resistors 50V ±100ppm/℃ ±1% 5.49kΩ 0402 C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, lib:R0402, F.Cu at (132.4, 132.1)
- added R75: 62.5mW Thick Film Resistors 50V ±100ppm/℃ ±1% 5.49kΩ 0402 C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, lib:R0402, F.Cu at (72.9, 134.5)
- added R76: 62.5mW Thick Film Resistors 50V ±100ppm/℃ ±1% 5.49kΩ 0402 C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, lib:R0402, F.Cu at (52.9, 139.1)
- added R77: 62.5mW Thick Film Resistors 50V ±100ppm/℃ ±1% 5.49kΩ 0402 C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, lib:R0402, F.Cu at (137.6, 134.3)
- added R78: 62.5mW Thick Film Resistors 50V ±100ppm/℃ ±1% 5.49kΩ 0402 C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, lib:R0402, F.Cu at (132.4, 130.0)
- added R79: 62.5mW Thick Film Resistors 50V ±100ppm/℃ ±1% 5.49kΩ 0402 C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, lib:R0402, F.Cu at (125.0, 139.1)
- added R8: 62.5mW Thick Film Resistors 50V ±100ppm/℃ ±1% 5.49kΩ 0402 C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, lib:R0402, F.Cu at (102.8, 132.2)
- added R80: 62.5mW Thick Film Resistors 50V ±100ppm/℃ ±1% 5.49kΩ 0402 C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, lib:R0402, F.Cu at (72.9, 132.2)
- added R81: 62.5mW Thick Film Resistors 50V ±100ppm/℃ ±1% 5.49kΩ 0402 C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, lib:R0402, F.Cu at (132.4, 139.1)
- added R82: 62.5mW Thick Film Resistors 50V ±100ppm/℃ ±1% 5.49kΩ 0402 C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, lib:R0402, F.Cu at (57.1, 139.1)
- added R83: 62.5mW Thick Film Resistors 50V ±100ppm/℃ ±1% 5.49kΩ 0402 C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, lib:R0402, F.Cu at (83.7, 130.0)
- added R84: 62.5mW Thick Film Resistors 50V ±100ppm/℃ ±1% 5.49kΩ 0402 C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, lib:R0402, F.Cu at (85.4, 136.8)
- added R85: 62.5mW Thick Film Resistors 50V ±100ppm/℃ ±1% 5.49kΩ 0402 C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, lib:R0402, F.Cu at (65.6, 130.0)
- added R86: 62.5mW Thick Film Resistors 50V ±100ppm/℃ ±1% 5.49kΩ 0402 C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, lib:R0402, F.Cu at (57.1, 130.0)
- added R87: 62.5mW Thick Film Resistors 50V ±100ppm/℃ ±1% 5.49kΩ 0402 C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, lib:R0402, F.Cu at (116.1, 136.8)
- added R88: 62.5mW Thick Film Resistors 50V ±100ppm/℃ ±1% 5.49kΩ 0402 C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, lib:R0402, F.Cu at (79.7, 134.0)
- added R89: 62.5mW Thick Film Resistors 50V ±100ppm/℃ ±1% 5.49kΩ 0402 C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, lib:R0402, F.Cu at (47.7, 130.0)
- added R9: 62.5mW Thick Film Resistors 50V ±100ppm/℃ ±1% 5.49kΩ 0402 C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, lib:R0402, F.Cu at (52.9, 136.8)
- added R90: 62.5mW Thick Film Resistors 50V ±100ppm/℃ ±1% 5.49kΩ 0402 C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, lib:R0402, F.Cu at (52.9, 134.5)
- added R91: 62.5mW Thick Film Resistors 50V ±100ppm/℃ ±1% 5.49kΩ 0402 C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, lib:R0402, F.Cu at (65.6, 134.5)
- added R92: 62.5mW Thick Film Resistors 50V ±100ppm/℃ ±1% 5.49kΩ 0402 C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, lib:R0402, F.Cu at (125.0, 136.8)
- added R93: 62.5mW Thick Film Resistors 50V ±100ppm/℃ ±1% 5.49kΩ 0402 C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, lib:R0402, F.Cu at (127.6, 139.1)
- added R94: 62.5mW Thick Film Resistors 50V ±100ppm/℃ ±1% 5.49kΩ 0402 C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, lib:R0402, F.Cu at (77.7, 139.1)
- added R95: 62.5mW Thick Film Resistors 50V ±100ppm/℃ ±1% 5.49kΩ 0402 C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, lib:R0402, F.Cu at (116.1, 132.2)
- added R96: 62.5mW Thick Film Resistors 50V ±100ppm/℃ ±1% 5.49kΩ 0402 C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, lib:R0402, F.Cu at (121.1, 139.1)
- added R97: 62.5mW Thick Film Resistors 50V ±100ppm/℃ ±1% 5.49kΩ 0402 C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, lib:R0402, F.Cu at (52.9, 132.2)
- added R98: 62.5mW Thick Film Resistors 50V ±100ppm/℃ ±1% 5.49kΩ 0402 C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, lib:R0402, F.Cu at (47.7, 134.5)
- added R99: 62.5mW Thick Film Resistors 50V ±100ppm/℃ ±1% 5.49kΩ 0402 C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, lib:R0402, F.Cu at (108.0, 139.1)
- added U1: ?, lib:USB-C-SMD_KH-TYPE-C-16P, F.Cu at (82.5, 173.1)
- added U2: ?, lib:SOT-23-3_L2.9-W1.3-P0.95-LS2.4-BR, F.Cu at (124.5, 167.4)
- added U3: ?, lib:WIRELM-SMD_ESP32-S3-WROOM-1, F.Cu at (107.4, 158.8)
- added U4: ?, lib:KEY-SMD_4P-L4.2-W3.2-P2.20-LS4.6, F.Cu at (120.6, 162.3)
Routing:
- net esp32.ic-vcc-1: track 0.00 -> 127.0 mm
- net 5V: track 0.00 -> 117.3 mm, vias 0 -> 158
- net dm: track 0.00 -> 57.9 mm, vias 0 -> 2
- net dp: track 0.00 -> 55.3 mm, vias 0 -> 2
- net esp32.ic-vcc: track 0.00 -> 40.4 mm
- net GND_HELLO_WORLD: track 0.00 -> 13.3 mm
- net 3V3: track 0.00 -> 11.5 mm
- net en: track 0.00 -> 8.40 mm
- net gnd: track 0.00 -> 8.02 mm
- net GND_LOGO: track 0.00 -> 4.22 mm
- net logo_switch.fet-gate: track 0.00 -> 3.15 mm
- net hello_world_switch.fet-gate: track 0.00 -> 2.76 mm
- net cc2: track 0.00 -> 1.65 mm
- net cc1: track 0.00 -> 1.60 mm
- net (no net): track 0.00 -> 1.21 mm
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- added copper zone on B.Cu, net 5V
- added copper zone on F.Cu, net GND_HELLO_WORLD
- added copper zone on F.Cu, net GND_LOGO
- added copper zone on F.Cu, net gnd
Other:
- board size 225.7 x 100.8 mm -> 105 x 88 mm
- board text added: "HELLO WORLD!"
- board text removed: "{{GITHASH}}"
